File: PCB/tester/main core.kicad_sch (KiCad schematic)
At the start: 44 parts, among them J2 Conn_02x03_Odd_Even, Q1 DMN63D8L-7, SW1 SW_SPST, SW2 SW_SPST, SW3 SW_SPST, SW4 SW_SPST, SW5 SW_SPST, SW6 SW_SPST, SW7 SW_SPST, SW8 SW_SPST, SW9 SW_SPST, U5 ATXMEGA32A4U-MH

Commit message: Red LED & decouplers
- decoupler dos Switches mudados posição
- LED vermelho & R_LED mudados valor/refª
Parts:
- D8: MPN VFHR1116P-4C82A-TR -> 5990010007F; OEPSPN OEPS030038 -> OEPS030044
- R17: value 10k -> 560R; MPN CPF0402B10KE1 -> CRCW0402560RFKED; OEPSPN OEPS020043 -> OEPS020193; Tolerance 0.1% -> 1%
Changed lines of the file:
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@@
 			)
 		)
-		(property "Value" "10k"
+		(property "Value" "560R"
 			(at 46.99 181.61 90)
 			(show_name no)
@@
 			)
 		)
-		(property "Description" "SMD 0402 10kΩ ±0.1% 0.063W"
+		(property "Description" "SMD 0402 560Ω ±1% 0.063W"
 			(at 46.99 185.42 0)
 			(hide yes)
@@
 			)
 		)
-		(property "MPN" "CPF0402B10KE1"
+		(property "MPN" "CRCW0402560RFKED"
 			(at 43.942 194.183 0)
 			(hide yes)
@@
 			)
 		)
-		(property "OEPSPN" "OEPS020043"
+		(property "OEPSPN" "OEPS020193"
 			(at 46.99 185.42 0)
 			(hide yes)
@@
 			)
 		)
-		(property "Tolerance" "0.1%"
+		(property "Tolerance" "1%"
 			(at 46.99 185.42 0)
 			(hide yes)
@@
 			)
 		)
-		(property "MPN" "VFHR1116P-4C82A-TR"
+		(property "MPN" "5990010007F"
 			(at 38.1 185.42 0)
 			(hide yes)
@@
 			)
 		)
-		(property "OEPSPN" "OEPS030038"
+		(property "OEPSPN" "OEPS030044"
 			(at 38.1 185.42 0)
 			(hide yes)
