File: PCB/tester/FED3 tester.kicad_sch (KiCad schematic)
At the start: 31 parts, among them J1 USB4105-GF-A, U1 FT232RL, U2 LP5907MFX-3.3, U3 LP5907MFX-3.3, U4 TPS73801DCQR

Commit message: promenores componentes para a BOM
Parts:
- C14: TempCo X5R -> X7R
- L1, L2: value 40R@100MHz -> MI0805K400R-10
- R7: value 8k2 -> 8.2k
- U1: value FT232RL -> FT232RNL-REEL
Changed lines of the file:
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@@
 			)
 		)
-		(property "TempCo" "X5R"
+		(property "TempCo" "X7R"
 			(at 95.25 160.02 0)
 			(hide yes)
@@
 			)
 		)
-		(property "Value" "FT232RL"
+		(property "Value" "FT232RNL-REEL"
 			(at 120.65 29.972 0)
 			(show_name no)
@@
 			)
 		)
-		(property "Value" "40R@100MHz"
+		(property "Value" "MI0805K400R-10"
 			(at 88.9 33.8836 90)
 			(show_name no)
@@
 			)
 		)
-		(property "Value" "8k2"
+		(property "Value" "8.2k"
 			(at 86.106 160.782 0)
 			(show_name no)
@@
 			)
 		)
-		(property "Value" "40R@100MHz"
+		(property "Value" "MI0805K400R-10"
 			(at 71.12 33.8836 90)
 			(show_name no)
