File: PCB/tester/FED3 tester.kicad_sch (KiCad schematic)
At the start: 31 parts, among them J1 USB4105-GF-A, U1 FT232RNL-REEL, U2 LP5907MFX-3.3, U3 LP5907MFX-3.3, U4 TPS73801DCQR

Commit message: sync with main
Parts:
- R1, R3: MPN ERJ-2RKF5101X -> RT0402BRD075K1L; OEPSPN OEPS020173 -> OEPS020203; Tolerance 1% -> 0.1%
Other:
- moved on the sheet: C3, R2
