File: PCB/tester/FED3 tester.kicad_sch (KiCad schematic)
At the start: 31 parts, among them J1 USB4105-GF-A, U1 FT232RNL-REEL, U2 LP5907MFX-3.3, U3 LP5907MFX-3.3, U4 TPS73801DCQR

Commit message: para revisão ao Filipe
Parts:
- R7: value 8.2k -> 6.8k; footprint Resistor_SMD:R_0603_1608Metric -> Resistor_SMD:R_0402_1005Metric; MPN ERJ-3EKF8201V -> RC0402FR-076K8L; OEPSPN OEPS020103 -> OEPS020242
Changed lines of the file:
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@@
 		(in_pos_files yes)
 		(dnp no)
-		(property "Reference" "#PWR07"
+		(property "Reference" "#PWR08"
 			(at 107.95 52.07 0)
 			(hide yes)
@@
 			(project "FED3 tester"
 				(path "/2ba63f12-2fcd-4471-9636-2762cde37de8"
-					(reference "#PWR07")
+					(reference "#PWR08")
 					(unit 1)
 				)
@@
 		(in_pos_files yes)
 		(dnp no)
-		(property "Reference" "#PWR08"
+		(property "Reference" "#PWR07"
 			(at 74.93 52.07 0)
 			(hide yes)
@@
 			(project "FED3 tester"
 				(path "/2ba63f12-2fcd-4471-9636-2762cde37de8"
-					(reference "#PWR08")
+					(reference "#PWR07")
 					(unit 1)
 				)
@@
 			)
 		)
-		(property "Value" "8.2k"
+		(property "Value" "6.8k"
 			(at 86.106 160.782 0)
 			(show_name no)
@@
 			)
 		)
-		(property "Footprint" "Resistor_SMD:R_0603_1608Metric"
+		(property "Footprint" "Resistor_SMD:R_0402_1005Metric"
 			(at 88.646 159.766 90)
 			(hide yes)
@@
 			)
 		)
-		(property "Description" "RESISTOR:   SMD 0603 8.2kΩ ±1% 0.100W   [ERJ-3EKF8201V] [SMD]"
+		(property "Description" "RESISTOR:   SMD 0402 6.8kΩ ±1% 0.063W"
 			(at 87.63 160.02 0)
 			(hide yes)
@@
 			)
 		)
-		(property "MPN" "ERJ-3EKF8201V"
+		(property "MPN" "RC0402FR-076K8L"
 			(at 78.867 163.068 0)
 			(hide yes)
@@
 			)
 		)
-		(property "OEPSPN" "OEPS020103"
+		(property "OEPSPN" "OEPS020242"
 			(at 87.63 160.02 0)
 			(hide yes)
@@
 	)
 	(embedded_fonts no)
-	(embedded_files
-		(file
-			(name "generic.kicad_wks")
-			(type worksheet)
-			(data |KLUv/WDdCX0VAPbdXiHwth4UjMf84wQpaKiddXNyw2vE3ASpJOKm/UZkMyvPewFVAE4AWAA71P+6
-				E/V/PHhP6hl7NhdyvnNBg6Vy+uc/TLoZgwYrqd8THr90vwAABASi6O845VVxKvxdDihWvvVz++br
-				MViUUkSd1bPG476jAiAgGEMkzsd5OFQI1UctVrTy7u1E2OrTmkrby9ifu+L1uW/e2nvQp88q5Gmw
-				8ws+fr+f9y+L9Oa88s83DLU3p1VMWf3Lt9ZppVX9shLSUuq/uR+rym/I5fdulhPePlB3nqiaJruM
-				7sWyKo9QmUhQSqlo2yXTcBxYQ4ugCHXaOS+p8GvKeqUyDObgZJlt01AEZ9znHHtv076fr+emDv5R
-				BLLVKWaq1mfXdZMiCoDPukPdBgGBofrisvaiijoRFEPJJqbMiaFuzLqhYJZJpTHlApNlkM2yEDIx
-				wSiZRHvgh4dB7rEbqteFnDSTYDQM+BhzSVrph/3v/WyDQ2rwaZU/F27d8X1FznLJLFiAhKDhRMcY
-				khEJkiRJOnBEpOSqG67IIUSIB6wVkypOj83iBj0zp4LL2kMMw+lEgMAIPplQr3guKCdlw/SfU9Pm
-				wv5Qjf2c0i+iukyGwJWg6H+jq3g9lh1bbaelmbDHUSOcHe0f4IqIU3pYnNopN2UGuqm6tUzbD0DL
-				A846XZ/tXUnW1CdqEKGhzI4PDvNZEWdNQVTqjKoxCJiOkLlyPnE2aN0Mgntwtl4Il0TKJW3CO+mz
-				Z3UY05BTT9QUnWnIY2O5jqbO0VBDfwAQ0J2lPShW8OIwbtD7c16HHQWSRlikdRdv3bO2EHlrLTcN
-				okDmqiZIAfyy8oU9FMxL3Rl0kbp+k4D31UmB0+QSWL73QeUaK7tJbNu8DHaE+JnfMeyjQJuerxNn
-				/RsMH2E/mWuAPwa9Cg==|
-			)
-			(checksum "29ED9DE70340A48902A32D9A43F096A1")
-		)
-	)
 )
