File: PCB/tester/DUT.kicad_sch (KiCad schematic)
At the start: 72 parts, among them J3 6pin_hd, J4 61300621021, J5 PPTC051LFBN-RC, J6 61300511021, J7 PPTC021LFBN-RC, K1 Relay SPDT, K2 Relay SPDT, K3 Relay SPDT, Q2 PMF170XP,115, Q3 DMN63D8L-7, Q4 DMN63D8L-7, Q5 DMN63D8L-7, Q6 DMN63D8L-7, U6 THS4281, U7 THS4281, U8 THS4281, U9 ZXCT1082

Commit message: para revisão ao Filipe
Parts:
- removed R37: 5k, Resistor_SMD:R_0402_1005Metric, symbol Device:R_US
- removed R44: 24k, Resistor_SMD:R_0402_1005Metric, symbol Device:R_US
- removed R45, R49: 249k, Resistor_SMD:R_0402_1005Metric, symbol Device:R_US
- removed R47: 4.3k, Resistor_SMD:R_0603_1608Metric, symbol Device:R_US
- removed U9: ZXCT1082, Package_TO_SOT_SMD:SOT-23-5, symbol FED3 SymbLib:ZXC1082
- added C38: 100nF, Capacitor_SMD:C_0402_1005Metric, symbol Device:C_Small
- added R33: 1R, Resistor_SMD:R_0603_1608Metric, symbol Device:R_US
- added U9: INA214AI, Package_TO_SOT_SMD:SOT-363_SC-70-6, symbol FED3 SymbLib:INA214AI
- R35: renamed from R33; value 0.5R -> 1R; footprint Resistor_SMD:R_0805_2012Metric -> Resistor_SMD:R_0603_1608Metric; MPN RL1220S-R50-F -> RT0603BRD071RL; OEPSPN OEPS020221 -> OEPS020243; Tolerance 1% -> 0.1%
- R39: renamed from R36; value 5k -> 15R; footprint Resistor_SMD:R_0402_1005Metric -> Resistor_SMD:R_1206_3216Metric; MPN PNM0402E5001BST1 -> PHPA1206E15R0BST1; OEPSPN OEPS020206 -> OEPS020244
- renumbered D11 to D10, D9 to D11, D10 to D9, K2 to K1, K3 to K2, K1 to K3, Q6 to Q4, Q4 to Q6, R46 to R34, R34 to R36, R48 to R37, R43 to R42, R35 to R43, R39 to R44, R42 to R45
Connections:
- net +3V3: now also C38.1, U9.3 (Vcc); no longer J3.6 (Pin_6), J4.1 (Pin_1)
- net Bat I ADC : now also U9.6 (OUT); no longer K2.3
- net GND: now also C38.2, U9.1 (REF), U9.2 (GND)
- net VBatt_DUT: now also R39.1, R33.2, U9.5 (IN-)
- net at K3.3, R43.2: now also K2.3, U9.4 (IN+); no longer R35.1, R39.2
- net at K2.5: now also R39.2
- net at K2.7: now also R35.1, R33.1
- no-connect marks 5 -> 4
Other:
- note added: "I=100uA"
- note added: "I=8.8mA"
- moved on the sheet: D10, D11, D9, J7, K1, K2, K3, Q4, Q5, Q6, R34, R35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

Commit message: redimensionamento mecânico & ficheiros produção
- FED3-tester & support redimensionadas mecanicamente, na zona onde ficará o ecrã de FED3
- pequenas correcções eléctricas vistas pelo Filipe
- gerados ficheiros de produção de acordo com "Procedure - Generate KiCAD productionfiles"
Connections:
- net +3V3: now also J4.1 (Pin_1)
- net GND: no longer J3.1 (Pin_1)
- no-connect marks 4 -> 6
Changed lines of the file:
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@@
 		(at 74.93 153.67)
 	)
+	(no_connect
+		(at 267.97 22.86)
+	)
+	(no_connect
+		(at 255.27 27.94)
+	)
 	(wire
 		(pts
@@
 	(wire
 		(pts
-			(xy 252.73 27.94) (xy 255.27 27.94)
-		)
-		(stroke
-			(width 0)
-			(type solid)
-		)
-	)
-	(wire
-		(pts
 			(xy 41.91 177.8) (xy 44.45 177.8)
 		)
@@
 	(wire
 		(pts
+			(xy 269.24 39.37) (xy 267.97 39.37)
+		)
+		(stroke
+			(width 0)
+			(type default)
+		)
+	)
+	(wire
+		(pts
 			(xy 144.78 72.39) (xy 144.78 71.12)
 		)
@@
 	(wire
 		(pts
+			(xy 269.24 36.83) (xy 269.24 39.37)
+		)
+		(stroke
+			(width 0)
+			(type default)
+		)
+	)
+	(wire
+		(pts
 			(xy 256.54 60.96) (xy 260.35 60.96)
 		)
@@
 	(symbol
 		(lib_id "power:GNDD")
-		(at 252.73 27.94 0)
-		(unit 1)
-		(body_style 1)
-		(exclude_from_sim no)
-		(in_bom yes)
-		(on_board yes)
-		(in_pos_files yes)
-		(dnp no)
-		(property "Reference" "#PWR073"
-			(at 252.73 27.94 0)
-			(hide yes)
-			(show_name no)
-			(do_not_autoplace no)
-			(effects
-				(font
-					(size 1.27 1.27)
-				)
-				(justify bottom)
-			)
-		)
-		(property "Value" "GND"
-			(at 252.73 32.766 0)
-			(show_name no)
-			(do_not_autoplace no)
-			(effects
-				(font
-					(size 1.27 1.27)
-				)
-				(justify bottom)
-			)
-		)
-		(property "Footprint" ""
-			(at 252.73 27.94 0)
-			(hide yes)
-			(show_name no)
-			(do_not_autoplace no)
-			(effects
-				(font
-					(size 1.27 1.27)
-				)
-			)
-		)
-		(property "Datasheet" ""
-			(at 252.73 27.94 0)
-			(hide yes)
-			(show_name no)
-			(do_not_autoplace no)
-			(effects
-				(font
-					(size 1.27 1.27)
-				)
-			)
-		)
-		(property "Description" "Power symbol creates a global label with name \"GNDD\" , digital ground"
-			(at 252.73 27.94 0)
-			(hide yes)
-			(show_name no)
-			(do_not_autoplace no)
-			(effects
-				(font
-					(size 1.27 1.27)
-				)
-			)
-		)
-		(pin "1"
-		)
-		(instances
-			(project "FED3 tester"
-				(path "/2ba63f12-2fcd-4471-9636-2762cde37de8/a050073c-fe8b-47ad-8c37-c2ab8f59b63a/838e2ae2-22cc-4dd4-86ab-e15afb1cdb8d"
-					(reference "#PWR073")
-					(unit 1)
-				)
-			)
-		)
-	)
-	(symbol
-		(lib_id "power:GNDD")
 		(at 35.56 142.24 0)
 		(unit 1)
@@
 					(unit 1)
 				)
+			)
+		)
+	)
+	(symbol
+		(lib_id "power:+3V3")
+		(at 269.24 36.83 0)
+		(unit 1)
+		(body_style 1)
+		(exclude_from_sim no)
+		(in_bom yes)
+		(on_board yes)
+		(in_pos_files yes)
+		(dnp no)
+		(property "Reference" "#PWR073"
+			(at 269.24 40.64 0)
+			(hide yes)
+			(show_name no)
+			(do_not_autoplace no)
+			(effects
+				(font
+					(size 1.27 1.27)
+				)
+			)
+		)
+		(property "Value" "+3V3"
+			(at 268.478 32.766 0)
+			(show_name no)
+			(do_not_autoplace no)
+			(effects
+				(font
+					(size 1.27 1.27)
+				)
+			)
+		)
+		(property "Footprint" ""
+			(at 269.24 36.83 0)
+			(hide yes)
+			(show_name no)
+			(do_not_autoplace no)
+			(effects
+				(font
+					(size 1.27 1.27)
+				)
+			)
+		)
+		(property "Datasheet" ""
+			(at 269.24 36.83 0)
+			(hide yes)
+			(show_name no)
+			(do_not_autoplace no)
+			(effects
+				(font
+					(size 1.27 1.27)
+				)
+			)
+		)
+		(property "Description" "Power symbol creates a global label with name \"+3V3\""
+			(at 269.24 36.83 0)
+			(hide yes)
+			(show_name no)
+			(do_not_autoplace no)
+			(effects
+				(font
+					(size 1.27 1.27)
+				)
+			)
+		)
+		(pin "1"
+		)
+		(instances
+			(project "FED3 tester"
+				(path "/2ba63f12-2fcd-4471-9636-2762cde37de8/a050073c-fe8b-47ad-8c37-c2ab8f59b63a/838e2ae2-22cc-4dd4-86ab-e15afb1cdb8d"
+					(reference "#PWR073")
+					(unit 1)
+				)
