File: PCB/tester/FED3 tester.kicad_pcb (KiCad board)
At the start: 4 copper layers, 108 x 134.4 mm, 163 parts, among them J1 USB4105-GF-A, J2 PR20203VBDN, J3 6pin_hd, J4 61300621021, J5 PPTC051LFBN-RC, J6 61300511021, J7 PPTC021LFBN-RC, K1 Relay SPDT, K2 Relay SPDT, K3 Relay SPDT, Q1 DMN63D8L-7, Q2 PMF170XP,115, Q3 DMN63D8L-7, Q4 DMN63D8L-7, Q5 DMN63D8L-7, Q6 DMN63D8L-7, SW1 TL3305BF260QG, SW2 TL3305BF260QG, SW3 TL3305BF260QG, SW4 TL3305BF260QG, SW5 TL3305BF260QG, SW6 TL3305BF260QG, SW7 TL3305BF260QG, SW8 TL3305BF260QG, SW9 TL3305BF260QG, U1 FT232RNL-REEL, U2 LP5907MFX-3.3, U3 LP5907MFX-3.3, U4 TPS73801DCQR, U5 ATXMEGA32A4U-MH, U6 THS4281, U7 THS4281, U8 THS4281, U9 INA214AI

Commit message: redimensionamento mecânico & ficheiros produção
- FED3-tester & support redimensionadas mecanicamente, na zona onde ficará o ecrã de FED3
- pequenas correcções eléctricas vistas pelo Filipe
- gerados ficheiros de produção de acordo com "Procedure - Generate KiCAD productionfiles"
Parts:
- removed the ? at (158.0, 30.6)
Connections:
- J3 pad 1: GND -> unconnected-(J3-Pin_1-Pad1)
- J4 pad 1: unconnected-(J4-Pin_1-Pad1) -> +3V3
Routing:
- net +3V3: track 535.2 -> 628.9 mm, vias 21 -> 22
- net GND: vias 238 -> 237
Other:
- board size 108 x 134.4 mm -> 104.8 x 134.4 mm
Changed lines of the file:
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@@
 		)
 	)
-	(footprint "FED3_PCBLib:MechHole_7mm"
-		(layer "F.Cu")
-		(at 158.02 30.56)
-		(property "Reference" ""
-			(at 0 -0.5 0)
-			(unlocked yes)
-			(layer "F.SilkS")
-			(hide yes)
-			(effects
-				(font
-					(size 1 1)
-					(thickness 0.2)
-				)
-			)
-		)
-		(property "Value" "MechHole_7mm"
-			(at 0 1 0)
-			(unlocked yes)
-			(layer "F.Fab")
-			(hide yes)
-			(effects
-				(font
-					(size 1 1)
-					(thickness 0.15)
-				)
-			)
-		)
-		(property "Datasheet" ""
-			(at 0 0 0)
-			(unlocked yes)
-			(layer "F.Fab")
-			(hide yes)
-			(effects
-				(font
-					(size 1 1)
-					(thickness 0.15)
-				)
-			)
-		)
-		(property "Description" ""
-			(at 0 0 0)
-			(unlocked yes)
-			(layer "F.Fab")
-			(hide yes)
-			(effects
-				(font
-					(size 1 1)
-					(thickness 0.15)
-				)
-			)
-		)
-		(attr board_only exclude_from_pos_files exclude_from_bom)
-		(duplicate_pad_numbers_are_jumpers no)
-		(fp_circle
-			(center 0 0)
-			(end 0 4.4)
-			(stroke
-				(width 0.3)
-				(type solid)
-			)
-			(fill no)
-			(layer "F.SilkS")
-		)
-		(pad "" np_thru_hole circle
-			(at 0 0)
-			(size 1 1)
-			(drill 7)
-			(layers "*.Cu")
-			(clearance 1)
-		)
-		(embedded_fonts no)
-	)
 	(footprint "Capacitor_SMD:C_1206_3216Metric"
 		(layer "F.Cu")
@@
 			(layers "*.Cu" "*.Mask")
 			(remove_unused_layers no)
-			(net "GND")
+			(net "unconnected-(J3-Pin_1-Pad1)")
 			(pinfunction "Pin_1_1")
-			(pintype "passive")
+			(pintype "passive+no_connect")
 		)
 		(pad "2" thru_hole circle
@@
 			(net "unconnected-(J3-Pin_6-Pad6)")
 			(pinfunction "Pin_6_6")
-			(pintype "passive")
+			(pintype "passive+no_connect")
 		)
 		(embedded_fonts no)
@@
 			(layers "*.Cu" "*.Mask")
 			(remove_unused_layers no)
-			(net "unconnected-(J4-Pin_1-Pad1)")
+			(net "+3V3")
 			(pinfunction "Pin_1_1")
 			(pintype "passive")
@@
 		(embedded_fonts no)
 		(model "${KIPRJMOD}/FED3_PCBLib.pretty/FED3_v7.3 v2.step"
-			(hide yes)
-			(opacity 0.3500)
+			(opacity 0.5900)
 			(offset
 				(xyz -0.5 0 -12)
@@
 		(layer "Eco2.User")
 	)
-	(gr_circle
-		(center 158.02 30.56)
-		(end 157.21 30.56)
-		(stroke
-			(width 0.1)
-			(type default)
-		)
-		(fill no)
-		(layer "Eco2.User")
-	)
 	(gr_line
 		(start 56.72 29.16)
@@
 	(gr_line
 		(start 123.72 24.16)
-		(end 159.72 24.16)
+		(end 152.92 24.16)
+		(stroke
+			(width 0.25)
+			(type solid)
+		)
+		(layer "Edge.Cuts")
+	)
+	(gr_line
+		(start 152.916419 34.9)
+		(end 161.5 34.9)
 		(stroke
 			(width 0.25)
@@
 	)
 	(gr_line
-		(start 159.72 24.16)
-		(end 164.72 29.16)
+		(start 152.92 24.16)
+		(end 152.916419 34.9)
 		(stroke
 			(width 0.25)
@@
 	)
 	(gr_line
-		(start 159.72 74.11)
+		(start 159.72 74.205833)
 		(end 159.72 158.52)
 		(stroke
@@
 	)
 	(gr_line
-		(start 164.72 29.16)
-		(end 164.72 69.11)
+		(start 161.5 34.9)
+		(end 161.5 72.5)
 		(stroke
 			(width 0.25)
@@
 	)
 	(gr_line
-		(start 164.72 69.11)
-		(end 159.72 74.11)
+		(start 161.5 72.5)
+		(end 159.72 74.205833)
 		(stroke
 			(width 0.25)
@@
 	)
 	(gr_text "GND"
-		(at 161.1 64.8 0)
+		(at 160.1 56.8 90)
 		(layer "F.SilkS")
 		(effects
@@
 	)
 	(via
-		(at 162.89 32.05)
+		(at 159.9 36.5)
 		(size 0.5)
 		(drill 0.2)
@@
 	)
 	(via
-		(at 162.93 51.7)
-		(size 0.5)
-		(drill 0.2)
-		(layers "F.Cu" "B.Cu")
-		(net "GND")
-	)
-	(via
 		(at 105.95 43.09)
 		(size 0.5)
@@
 	)
 	(via
-		(at 162.79 68.54)
+		(at 159.8 70.15)
 		(size 0.5)
 		(drill 0.2)
@@
 	)
 	(via
-		(at 157.18 25.7)
+		(at 151.3 26.2)
 		(size 0.5)
 		(drill 0.2)
@@
 	)
 	(via
-		(at 162.93 42.27)
+		(at 160.4 50.7)
 		(size 0.5)
 		(drill 0.2)
@@
 	)
 	(via
+		(at 108.15 78.7)
+		(size 0.5)
+		(drill 0.2)
+		(layers "F.Cu" "B.Cu")
+		(net "+3V3")
+	)
+	(via
 		(at 87 128.95)
 		(size 0.5)
@@
 	)
 	(segment
+		(start 107.82 79.08)
+		(end 107.82 148.57)
+		(width 0.22)
+		(layer "In1.Cu")
+		(net "+3V3")
+	)
+	(segment
+		(start 107.82 148.57)
+		(end 110.7 151.45)
+		(width 0.22)
+		(layer "In1.Cu")
+		(net "+3V3")
+	)
+	(segment
+		(start 110.7 151.45)
+		(end 110.7 151.820289)
+		(width 0.22)
+		(layer "In1.Cu")
+		(net "+3V3")
+	)
+	(segment
+		(start 108.15 78.75)
+		(end 107.82 79.08)
+		(width 0.22)
+		(layer "In1.Cu")
+		(net "+3V3")
+	)
+	(segment
+		(start 108.15 78.7)
+		(end 108.15 78.75)
+		(width 0.22)
+		(layer "In1.Cu")
+		(net "+3V3")
+	)
+	(segment
 		(start 146.15 77.45)
 		(end 145.6 78)
@@
 	)
 	(segment
+		(start 89.09 78.7)
+		(end 89.01 78.78)
+		(width 0.22)
+		(layer "In2.Cu")
+		(net "+3V3")
+	)
+	(segment
 		(start 87.56 67.21)
 		(end 130.02 67.21)
@@
 	)
 	(segment
+		(start 108.15 78.7)
+		(end 89.09 78.7)
+		(width 0.22)
+		(layer "In2.Cu")
+		(net "+3V3")
+	)
+	(segment
 		(start 86.615 33.785)
 		(end 125.52 33.785)
@@
 	)
 	(zone
-		(net "GND")
-		(layers "B.Cu" "In1.Cu" "In2.Cu")
-		(hatch edge 0.5)
-		(priority 2)
-		(connect_pads
-			(clearance 0.5)
-		)
-		(min_thickness 0.5)
-		(fill yes
-			(thermal_gap 0.5)
-			(thermal_bridge_width 0.5)
-			(island_removal_mode 0)
-		)
-		(polygon
-			(pts
-				(xy 158.375 74.04) (xy 163.375 69.04) (xy 163.375 30.25) (xy 158.375 25.25)
-			)
-		)
-	)
-	(zone
 		(layers "B.Cu" "In1.Cu" "In2.Cu")
 		(hatch edge 0.5)
@@
 		(polygon
 			(pts
-				(xy 63.95 25.25) (xy 63.95 157.6) (xy 158.375 157.6) (xy 158.375 25.25)
+				(xy 151.9 25.3) (xy 63.95 25.25) (xy 63.95 157.6) (xy 158.9 157.5) (xy 158.8 73.6) (xy 160.5 71.8)
+				(xy 160.9 35.4) (xy 151.9 35.4)
 			)
 		)
