File: PCB/support/FED3 tester - support.kicad_pcb (KiCad board)
At the start: 2 copper layers, 108 x 134.3 mm, 31 parts, among them J2 6pin_hd

Commit message: redimensionamento mecânico & ficheiros produção
- FED3-tester & support redimensionadas mecanicamente, na zona onde ficará o ecrã de FED3
- pequenas correcções eléctricas vistas pelo Filipe
- gerados ficheiros de produção de acordo com "Procedure - Generate KiCAD productionfiles"
Connections:
- J2 pad 6: +3V3 -> (no net)
Other:
- board size 108 x 134.3 mm -> 104.8 x 134.3 mm
- board text added: "FED3 tester - support rev.C"
- board text removed: "FED3 tester - support rev.B"
Changed lines of the file:
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@@
 			(layers "*.Cu" "*.Mask")
 			(remove_unused_layers no)
-			(net "+3V3")
 			(pinfunction "Pin_6")
 			(pintype "passive")
@@
 	)
 	(gr_line
+		(start 112.3 37.84)
+		(end 141.5 37.84)
+		(stroke
+			(width 0.25)
+			(type solid)
+		)
+		(layer "Eco2.User")
+	)
+	(gr_line
+		(start 141.496419 48.58)
+		(end 150.08 48.58)
+		(stroke
+			(width 0.25)
+			(type solid)
+		)
+		(layer "Eco2.User")
+	)
+	(gr_line
+		(start 141.5 37.84)
+		(end 141.496419 48.58)
+		(stroke
+			(width 0.25)
+			(type solid)
+		)
+		(layer "Eco2.User")
+	)
+	(gr_line
+		(start 148.3 87.885833)
+		(end 148.3 172.2)
+		(stroke
+			(width 0.25)
+			(type solid)
+		)
+		(layer "Eco2.User")
+	)
+	(gr_line
+		(start 148.3 172.2)
+		(end 131.15 172.2)
+		(stroke
+			(width 0.25)
+			(type solid)
+		)
+		(layer "Eco2.User")
+	)
+	(gr_line
+		(start 150.08 48.58)
+		(end 150.08 86.18)
+		(stroke
+			(width 0.25)
+			(type solid)
+		)
+		(layer "Eco2.User")
+	)
+	(gr_line
+		(start 150.08 86.18)
+		(end 148.3 87.885833)
+		(stroke
+			(width 0.25)
+			(type solid)
+		)
+		(layer "Eco2.User")
+	)
+	(gr_line
 		(start 45.3 42.856049)
 		(end 50.3 37.856049)
@@
 	(gr_line
 		(start 148.3 37.856049)
-		(end 153.3 42.856049)
+		(end 150.1 39.656049)
 		(stroke
 			(width 0.25)
@@
 	)
 	(gr_line
-		(start 153.3 42.856049)
-		(end 153.3 82.806049)
-		(stroke
-			(width 0.25)
-			(type solid)
-		)
-		(layer "Edge.Cuts")
-	)
-	(gr_line
-		(start 153.3 82.806049)
+		(start 150.1 39.656049)
+		(end 150.1 86.18)
+		(stroke
+			(width 0.25)
+			(type solid)
+		)
+		(layer "Edge.Cuts")
+	)
+	(gr_line
+		(start 150.1 86.18)
 		(end 148.3 87.806049)
 		(stroke
@@
 		(layer "F.Fab")
 	)
-	(gr_text "FED3 tester - support\nrev.B"
+	(gr_text "FED3 tester - support\nrev.C"
 		(at 55 155.9 0)
 		(layer "F.SilkS")
@@
 		(members "957468f4-e4ee-485a-b667-6ad02b729629" "accb8aa6-8b86-4b77-aa7d-73aaa8904214")
 	)
+	(group ""
+		(members "4598e8d1-b6e9-4619-bb9f-74ffffb51fd7" "4b0b7326-fe85-4817-8006-6fe4922581e2"
+			"5965d3f2-d348-4256-b61b-e3e89064125d" "b4ca0044-781c-4b9a-b6bf-251304818474"
+			"bd3cd5bf-0add-429b-9e34-8926a9e5f62e" "e2bb4cec-dd85-46ea-98a4-904d53919b5c"
+			"ea84051f-5be9-4555-ae18-f53a7f7336e2"
+		)
+	)
 	(embedded_fonts no)
